Commit message: Modifications for FT mecanum basic

File: linorobot2_description/urdf/mecanum_properties.urdf.xacro (robot description, xacro)
@@ -1,20 +1,20 @@
 <?xml version="1.0"?>
 <robot xmlns:xacro="http://ros.org/wiki/xacro">
-  <xacro:property name="base_length" value="0.445" />
-  <xacro:property name="base_width" value="0.200" />
-  <xacro:property name="base_height" value="0.129" />
-  <xacro:property name="base_mass" value="10" />
-  <xacro:property name="wheel_radius" value="0.07162" />
-  <xacro:property name="wheel_width" value="0.05" />
-  <xacro:property name="wheel_pos_x" value="0.120" />
-  <xacro:property name="wheel_pos_y" value="0.1355" />
-  <xacro:property name="wheel_pos_z" value="-0.04788" />
+  <xacro:property name="base_length" value="0.4" />
+  <xacro:property name="base_width" value="0.26" />
+  <xacro:property name="base_height" value="0.4" />
+  <xacro:property name="base_mass" value="50" />
+  <xacro:property name="wheel_radius" value="0.076" />
+  <xacro:property name="wheel_width" value="0.056" />
+  <xacro:property name="wheel_pos_x" value="0.15" />
+  <xacro:property name="wheel_pos_y" value="0.183" />
+  <xacro:property name="wheel_pos_z" value="-0.40" />
   <xacro:property name="wheel_mass" value=".6" />
   <xacro:property name="wheel_torque" value="20" />
   <xacro:property name="laser_pose">
-    <origin xyz="-0.0475 0 0.125" rpy="0 0 0"/>
+    <origin xyz="0 0 0.575" rpy="0 0 0"/>
   </xacro:property>
   <xacro:property name="depth_sensor_pose">
-    <origin xyz="0.2375 0 0.06" rpy="0 0 0"/>
+    <origin xyz="0.225 0 0.1" rpy="0 0 0"/>
   </xacro:property>
 </robot>

Commit message: Fised issue with 2d Laser plugin

File: linorobot2_description/urdf/mecanum_properties.urdf.xacro (robot description, xacro)
@@ -3,5 +3,5 @@
   <xacro:property name="base_length" value="0.4" />
   <xacro:property name="base_width" value="0.26" />
-  <xacro:property name="base_height" value="0.4" />
+  <xacro:property name="base_height" value="0.8" />
   <xacro:property name="base_mass" value="50" />
   <xacro:property name="wheel_radius" value="0.076" />

Commit message: Added extra 2d lidar.

File: linorobot2_description/urdf/mecanum_properties.urdf.xacro (robot description, xacro)
@@ -15,4 +15,10 @@
     <origin xyz="0 0 0.575" rpy="0 0 0"/>
   </xacro:property>
+  <xacro:property name="base_f_laser_pose">
+    <origin xyz="0.25 0 -0.35" rpy="0 0 0"/>
+  </xacro:property>
+  <xacro:property name="base_r_laser_pose">
+    <origin xyz="-0.25 0 -0.35" rpy="0 0 3.1416"/>
+  </xacro:property>
   <xacro:property name="depth_sensor_pose">
     <origin xyz="0.225 0 0.1" rpy="0 0 0"/>

File: linorobot2_description/urdf/robots/mecanum.urdf.xacro (robot description, xacro)
@@ -56,4 +56,10 @@
     <xacro:insert_block name="laser_pose" />
   </xacro:generic_laser>
+  <xacro:generic_base_f_laser>
+    <xacro:insert_block name="base_f_laser_pose" />
+  </xacro:generic_base_f_laser>
+  <xacro:generic_base_r_laser>
+    <xacro:insert_block name="base_r_laser_pose" />
+  </xacro:generic_base_r_laser>
   <xacro:depth_sensor>
     <xacro:insert_block name="depth_sensor_pose" />

File: linorobot2_description/urdf/sensors/generic_laser.urdf.xacro (robot description, xacro)
@@ -16,14 +16,28 @@
     </xacro:laser>
   </xacro:macro>
-  <xacro:macro name="generic_base_laser" params="*origin">
+  <xacro:macro name="generic_base_f_laser" params="*origin">
     <xacro:laser
       update_rate="10"
       ray_count="360"
-      min_angle="-3.1416"
-      max_angle="3.1416"
+      min_angle="-1.57079632679"
+      max_angle="1.57079632679"
       min_range="0.21"
       max_range="5.5"
-      frame_id="base_laser"
-      topic_name="base/scan"
+      frame_id="base_laser_f"
+      topic_name="base/scan/f"
+    >
+      <xacro:insert_block name="origin" />
+    </xacro:laser>
+  </xacro:macro>
+  <xacro:macro name="generic_base_r_laser" params="*origin">
+    <xacro:laser
+      update_rate="10"
+      ray_count="360"
+      min_angle="-1.57079632679"
+      max_angle="1.57079632679"
+      min_range="0.21"
+      max_range="5.5"
+      frame_id="base_laser_r"
+      topic_name="base/scan/r"
     >
       <xacro:insert_block name="origin" />

File: linorobot2_description/urdf/sensors/laser.urdf.xacro (robot description, xacro)
@@ -46,5 +46,5 @@
         <update_rate>${update_rate}</update_rate>
         <pose>0 0 0 0 0 0</pose>
-        <visualize>true</visualize>
+        <visualize>false</visualize>
         <ray>
           <scan>
